Commit message: Update: unity上のic120を動かす際の設定を何点か修正

File: ic120_description/urdf/ic120_.xacro (robot description, xacro)
@@ -3,5 +3,4 @@
 	<xacro:property name="PI" value="3.1415926535" />
 	<xacro:property name="tf_prefix" value=""/>
-    <xacro:property name="ic120_description_dir_path" value=""/>
     <!-- Base Link -->
     <link name="${tf_prefix}/base_link"/>
@@ -14,6 +13,4 @@
             <geometry>
                 <mesh filename="package://ic120_description/meshes/ic120-body.dae"/>
-                <!-- <mesh filename="${ic120_description_dir_path}/meshes/ic120-body.dae"/> -->
-                <!-- <mesh filename="/home/common/SIP_PROJECTS/M2/DEV_TS/ros2_ws/install/ic120_description/share/ic120_description/meshes/ic120-body.dae"/> -->
             </geometry>
         </visual>
@@ -27,5 +24,5 @@
     </link>
     <!-- left sprocket axis -->
-    <joint name="${ic120_description_dir_path}sprocket_left_joint" type="continuous">
+    <joint name="sprocket_left_joint" type="continuous">
         <origin xyz="-2.35 1 0.65"/>
         <axis xyz="0 1 0"/>
