Commit message: Update some files

File: ic120_description/urdf/ic120.xacro (robot description, xacro)
@@ -5,8 +5,8 @@
 	<!-- <xacro:include filename="$(find ic120_description)/urdf/materials.xacro" /> -->
 	<!-- Base Link -->
-	<link name="base_link"/>
+	<link name="/base_link"/>
 	<joint name="base_joint" type="fixed">
-		<parent link="base_link"/>
-		<child link="body_link"/>
+		<parent link="/base_link"/>
+		<child link="/body_link"/>
 	</joint>
 	<link name="body_link">

Commit message: Update some files

File: ic120_description/urdf/ic120.xacro (robot description, xacro)
@@ -5,10 +5,10 @@
 	<!-- <xacro:include filename="$(find ic120_description)/urdf/materials.xacro" /> -->
 	<!-- Base Link -->
-	<link name="/base_link"/>
+	<link name="ic120_tf/base_link"/>
 	<joint name="base_joint" type="fixed">
-		<parent link="/base_link"/>
-		<child link="/body_link"/>
+		<parent link="ic120_tf/base_link"/>
+		<child link="ic120_tf/body_link"/>
 	</joint>
-	<link name="body_link">
+	<link name="ic120_tf/body_link">
 		<visual>
 			<geometry>
@@ -28,25 +28,25 @@
 		<origin xyz="-2.35 1 0.65"/>
 		<axis xyz="0 1 0"/>
-		<parent link="body_link"/>
-		<child link="left_sprocket_link"/>
+		<parent link="ic120_tf/body_link"/>
+		<child link="ic120_tf/left_sprocket_link"/>
 	</joint>
-	<link name="left_sprocket_link"/>
+	<link name="ic120_tf/left_sprocket_link"/>
 	<!-- right sprocket axis -->
 	<joint name="sprocket_right_joint" type="continuous">
 		<origin xyz="-2.35 -1 0.65"/>
 		<axis xyz="0 1 0"/>
-		<parent link="body_link"/>
-		<child link="right_sprocket_link"/>
+		<parent link="ic120_tf/body_link"/>
+		<child link="ic120_tf/right_sprocket_link"/>
 	</joint>
-	<link name="right_sprocket_link"/>
+	<link name="ic120_tf/right_sprocket_link"/>
 	<!-- bucket axis -->
 	<joint name="vessel_pin_joint" type="revolute">
 		<origin xyz="-3.0153 0 0.94605"/>
 		<axis xyz="0 1 0"/>
-		<parent link="body_link"/>
-		<child link="vessel_pin_link"/>
+		<parent link="ic120_tf/body_link"/>
+		<child link="ic120_tf/vessel_pin_link"/>
 		<limit lower="${-radians(65)}" upper="0" effort="30" velocity="6.159937255"/>
 	</joint>
-	<link name="vessel_pin_link">
+	<link name="ic120_tf/vessel_pin_link">
 		<visual>
 			<geometry>
@@ -66,9 +66,9 @@
 		<origin xyz="-0.75792 0 0.73083"/>
 		<axis xyz="0 1 0"/>
-		<parent link="body_link"/>
-		<child link="cylinder_head_link"/>
+		<parent link="ic120_tf/body_link"/>
+		<child link="ic120_tf/cylinder_head_link"/>
 		<mimic joint="vessel_pin_joint" multiplier="${radians(5.72)/radians(-65)}"/>
 	</joint>
-	<link name="cylinder_head_link">
+	<link name="ic120_tf/cylinder_head_link">
 		<visual>
 			<geometry>
@@ -87,11 +87,11 @@
 	<joint name="cylinder_rod_prismatic_joint" type="prismatic">
 		<origin xyz="0 0 0"/>
-		<parent link="cylinder_head_link"/>
-		<child link="cylinder_rod_link"/>
+		<parent link="ic120_tf/cylinder_head_link"/>
+		<child link="ic120_tf/cylinder_rod_link"/>
 		<axis xyz="-1.4989 0 0.51788"/>
 		<limit lower="-1" upper="1" effort="30" velocity="6.159937255"/>
 		<mimic joint="vessel_pin_joint" multiplier="${0.8/radians(-65)}"/>
 	</joint>
-	<link name="cylinder_rod_link">
+	<link name="ic120_tf/cylinder_rod_link">
 		<visual>
 			<geometry>

Commit message: Fix: 実機操作時の設定を一部変更

File: ic120_description/urdf/ic120.xacro (robot description, xacro)
@@ -2,5 +2,5 @@
 <robot name="ic120" xmlns:xacro="http://www.ros.org/wiki/xacro">
 	<xacro:property name="PI" value="3.1415926535" />
-	<xacro:property name="tf_prefix" value=""/>
+	<xacro:property name="tf_prefix" value="ic120_tf"/>
     <xacro:property name="ic120_description_dir_path" value=""/>
     <!-- Base Link -->
